File: Hardware/Power.kicad_sch (KiCad schematic)
At the start: 36 parts, among them Q3 PMPB47XP, Q4 BC847, Q5 BC847, U10 AP1509-33SG-13, U7 LT6654BHS6-2.5-TRMPBF, U8 TLS4125D0EPV50XUMA1, U9 LM2903DR2G

Commit message: Clean up custom KiCad libraries
- Clean up the directory structure for KiCad custom libraries.
- Fix paths in KiCad schematic and pcb for symbols, footprints, and
3d models for custom libraries.
Parts:
- C29, C32: footprint Libs:EEH-AZK1E471B -> Capacitor_THT:EEH-AZK1E471B
- D4: footprint Libs:Low_Batt_LED -> LED_THT:LTL-307P
- L1: footprint Libs:SRP1265C-220M -> Inductor_SMD:SRP1265C-220M
- L2: footprint Libs:CLF12577NIT-470M-D -> Inductor_SMD:CLF12577NIT-470M-D
- Q3: footprint Libs:PMPB47XP -> Transistor_SMD:PMPB47XP
- U10: footprint Libs:AP1509-33SG-13 -> IC:AP1509-33SG-13
- U7: footprint Libs:LT6654BHS6-2.5-TRMPBF -> IC:LT6654BHS6-2.5-TRMPBF
- U8: footprint Libs:TLS4125D0EPV50XUMA1 -> IC:TLS4125D0EPV50XUMA1
Changed lines of the file:
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@@
   (title_block
     (title "Musical Doorbell")
-    (date "2022-01-06")
-    (rev "B")
+    (date "2022-01-09")
+    (rev "A")
     (company "Michael Lazernik")
   )
@@
       (effects (font (size 1.524 1.524)))
     )
-    (property "Footprint" "Libs:TLS4125D0EPV50XUMA1" (id 2) (at 71.12 125.984 0)
+    (property "Footprint" "IC:TLS4125D0EPV50XUMA1" (id 2) (at 71.12 125.984 0)
       (effects (font (size 1.524 1.524)) hide)
     )
@@
     (property "Reference" "L1" (id 0) (at 102.87 126.2126 90))
     (property "Value" "SRP1265C-220M" (id 1) (at 102.87 128.524 90))
-    (property "Footprint" "Libs:SRP1265C-220M" (id 2) (at 102.87 130.81 0)
+    (property "Footprint" "Inductor_SMD:SRP1265C-220M" (id 2) (at 102.87 130.81 0)
       (effects (font (size 1.27 1.27)) hide)
     )
@@
       (effects (font (size 1.524 1.524)))
     )
-    (property "Footprint" "Libs:AP1509-33SG-13" (id 2) (at 224.79 59.944 0)
+    (property "Footprint" "IC:AP1509-33SG-13" (id 2) (at 224.79 59.944 0)
       (effects (font (size 1.524 1.524)) hide)
     )
@@
       (effects (font (size 1.27 1.27)) (justify left))
     )
-    (property "Footprint" "Libs:EEH-AZK1E471B" (id 2) (at 184.15 66.04 0)
+    (property "Footprint" "Capacitor_THT:EEH-AZK1E471B" (id 2) (at 184.15 66.04 0)
       (effects (font (size 1.27 1.27)) hide)
     )
@@
     (property "Reference" "Q3" (id 0) (at 143.51 93.9546 90))
     (property "Value" "PMPB47XP" (id 1) (at 143.51 96.266 90))
-    (property "Footprint" "Libs:PMPB47XP" (id 2) (at 146.05 92.71 0)
+    (property "Footprint" "Transistor_SMD:PMPB47XP" (id 2) (at 146.05 92.71 0)
       (effects (font (size 1.27 1.27)) hide)
     )
@@
       (effects (font (size 1.27 1.27)) (justify right))
     )
-    (property "Footprint" "Libs:Low_Batt_LED" (id 2) (at 171.45 49.53 0)
+    (property "Footprint" "LED_THT:LTL-307P" (id 2) (at 171.45 49.53 0)
       (effects (font (size 1.27 1.27)) hide)
     )
@@
     (property "Reference" "L2" (id 0) (at 254 58.9026 90))
     (property "Value" "CLF12577NIT-470M-D" (id 1) (at 254 61.214 90))
-    (property "Footprint" "Libs:CLF12577NIT-470M-D" (id 2) (at 254 63.5 0)
+    (property "Footprint" "Inductor_SMD:CLF12577NIT-470M-D" (id 2) (at 254 63.5 0)
       (effects (font (size 1.27 1.27)) hide)
     )
@@
       (effects (font (size 1.27 1.27)) (justify left))
     )
-    (property "Footprint" "Libs:EEH-AZK1E471B" (id 2) (at 273.05 68.58 0)
+    (property "Footprint" "Capacitor_THT:EEH-AZK1E471B" (id 2) (at 273.05 68.58 0)
       (effects (font (size 1.27 1.27)) hide)
     )
@@
       (effects (font (size 1.524 1.524)))
     )
-    (property "Footprint" "Libs:LT6654BHS6-2.5-TRMPBF" (id 2) (at 66.04 43.434 0)
+    (property "Footprint" "IC:LT6654BHS6-2.5-TRMPBF" (id 2) (at 66.04 43.434 0)
       (effects (font (size 1.524 1.524)) hide)
     )

Commit message: Cleanup custom KiCad libraries
- Delete unneeded/unused files
- Cleanup symbol library files for custom libraries
Parts:
- L1: symbol SRP1265C-220M:SRP1265C-220M -> Doorbell_Inductor_SMD:SRP1265C-220M
- U10: symbol AP1509-33SG-13:AP1509-33SG-13 -> Doorbell_IC:AP1509-33SG-13
- U7: symbol LT6654BHS6-2.5-TRMPBF:LT6654BHS6-2.5-TRMPBF -> Doorbell_IC:LT6654BHS6-2.5-TRMPBF
- U9: symbol LM2903DR2G:LM2903DR2G -> Doorbell_IC:LM2903DR2G
Changed lines of the file:
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@@
     (pin "9")
   )
-  (symbol (lib_id "SRP1265C-220M:SRP1265C-220M") (at 102.87 130.81 270) (unit 1)
+  (symbol (lib_id "Doorbell_Inductor_SMD:SRP1265C-220M") (at 102.87 130.81 270) (unit 1)
     (in_bom yes) (on_board yes)
     (property "Reference" "L1" (id 0) (at 102.87 126.2126 90))
@@
     (pin "1")
   )
-  (symbol (lib_id "AP1509-33SG-13:AP1509-33SG-13") (at 224.79 66.04 0) (unit 1)
+  (symbol (lib_id "Doorbell_IC:AP1509-33SG-13") (at 224.79 66.04 0) (unit 1)
     (in_bom yes) (on_board yes)
     (property "Reference" "U10" (id 0) (at 224.79 54.4322 0)
@@
     (pin "2")
   )
-  (symbol (lib_id "LT6654BHS6-2.5-TRMPBF:LT6654BHS6-2.5-TRMPBF") (at 66.04 49.53 0) (unit 1)
+  (symbol (lib_id "Doorbell_IC:LT6654BHS6-2.5-TRMPBF") (at 66.04 49.53 0) (unit 1)
     (in_bom yes) (on_board yes)
     (property "Reference" "U7" (id 0) (at 66.04 40.4622 0)
@@
     (pin "6")
   )
-  (symbol (lib_id "LM2903DR2G:LM2903DR2G") (at 116.84 60.96 0) (mirror y) (unit 1)
+  (symbol (lib_id "Doorbell_IC:LM2903DR2G") (at 116.84 60.96 0) (mirror y) (unit 1)
     (in_bom yes) (on_board yes)
     (property "Reference" "U9" (id 0) (at 116.84 51.6382 0))
@@
     (pin "3")
   )
-  (symbol (lib_id "LM2903DR2G:LM2903DR2G") (at 116.84 82.55 0) (unit 2)
+  (symbol (lib_id "Doorbell_IC:LM2903DR2G") (at 116.84 82.55 0) (unit 2)
     (in_bom yes) (on_board yes)
     (property "Reference" "U9" (id 0) (at 116.84 73.2282 0))
@@
     (pin "7")
   )
-  (symbol (lib_id "LM2903DR2G:LM2903DR2G") (at 116.84 49.53 270) (unit 3)
+  (symbol (lib_id "Doorbell_IC:LM2903DR2G") (at 116.84 49.53 270) (unit 3)
     (in_bom yes) (on_board yes)
     (property "Reference" "U9" (id 0) (at 116.84 41.275 90))

Commit message: Switch to local libraries for KiCad schematic
- Move all KiCad schematic symbols into local libraries
- Fix KiCad schematic library links to point to local libraries
Parts:
- C20, C21, C22, C23, C24, C25, C26, C27, C28, C30, C31: symbol Device:C_Small -> Doorbell_Capacitor:C_Small
- C29, C32: symbol Device:CP_Small -> Doorbell_Capacitor:C_Polarized_Small
- D3, D5: symbol Device:D_Zener_Small -> Doorbell_Diode:D_Zener_Small
- D4: symbol Device:LED -> Doorbell_LED:LED
- D6: symbol Device:D_Schottky_Small -> Doorbell_Diode:D_Schottky_Small
- L2: symbol Device:L_Small -> Doorbell_Inductor_SMD:L_Small
- Q3: symbol Device:Q_PMOS_DGS -> Doorbell_Transistor_SMD:Q_PMOS_DGS
- Q4, Q5: symbol Transistor_BJT:BC847 -> Doorbell_Transistor_SMD:BC847
- R16, R17, R18, R19, R20, R21, R22, R23, R24, R25: symbol Device:R_Small -> Doorbell_Resistor:R_Small
- U8: symbol TLS4125D0EPV50XUMA1:TLS4125D0EPV50XUMA1 -> Doorbell_IC:TLS4125D0EPV50XUMA1

Commit message: Move KiCad global footprint and 3d models to local
- Move KiCad global footprint and 3d models to local directories
- Reassign footprints in KiCad schematic/PCB from global libraries to
  local libraries
- Reassign global 3d models to local 3d models for KiCad
- Update KiCad PCB with all local footprints
Parts:
- D6: footprint Diode_SMD:D_SMF -> Diode_SMD:V3FM12-M3_H
- Q4, Q5: footprint Package_TO_SOT_SMD:SOT-23 -> Transistor_SMD:SOT-23
- U9: footprint Package_SO:SOIC-8_3.9x4.9mm_P1.27mm -> IC:SOIC-8_3.9x4.9mm_P1.27mm
Changed lines of the file:
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@@
       (effects (font (size 1.27 1.27)) (justify left))
     )
-    (property "Footprint" "Diode_SMD:D_SMF" (id 2) (at 251.46 77.47 90)
+    (property "Footprint" "Diode_SMD:V3FM12-M3_H" (id 2) (at 251.46 77.47 90)
       (effects (font (size 1.27 1.27)) hide)
     )
@@
       (effects (font (size 1.27 1.27)) (justify left))
     )
-    (property "Footprint" "Package_TO_SOT_SMD:SOT-23" (id 2) (at 173.99 92.075 0)
+    (property "Footprint" "Transistor_SMD:SOT-23" (id 2) (at 173.99 92.075 0)
       (effects (font (size 1.27 1.27) italic) (justify left) hide)
     )
@@
     (property "Reference" "Q5" (id 0) (at 224.79 85.6488 90))
     (property "Value" "BC847" (id 1) (at 224.79 87.9602 90))
-    (property "Footprint" "Package_TO_SOT_SMD:SOT-23" (id 2) (at 222.885 88.9 0)
+    (property "Footprint" "Transistor_SMD:SOT-23" (id 2) (at 222.885 88.9 0)
       (effects (font (size 1.27 1.27) italic) (justify left) hide)
     )
@@
     (property "Reference" "U9" (id 0) (at 116.84 51.6382 0))
     (property "Value" "LM2903DR2G" (id 1) (at 116.84 53.9496 0))
-    (property "Footprint" "Package_SO:SOIC-8_3.9x4.9mm_P1.27mm" (id 2) (at 116.84 60.96 0)
+    (property "Footprint" "IC:SOIC-8_3.9x4.9mm_P1.27mm" (id 2) (at 116.84 60.96 0)
       (effects (font (size 1.27 1.27)) hide)
     )
@@
     (property "Reference" "U9" (id 0) (at 116.84 73.2282 0))
     (property "Value" "LM2903DR2G" (id 1) (at 116.84 75.5396 0))
-    (property "Footprint" "Package_SO:SOIC-8_3.9x4.9mm_P1.27mm" (id 2) (at 116.84 82.55 0)
+    (property "Footprint" "IC:SOIC-8_3.9x4.9mm_P1.27mm" (id 2) (at 116.84 82.55 0)
       (effects (font (size 1.27 1.27)) hide)
     )
@@
     (property "Reference" "U9" (id 0) (at 116.84 41.275 90))
     (property "Value" "LM2903DR2G" (id 1) (at 116.84 43.5864 90))
-    (property "Footprint" "Package_SO:SOIC-8_3.9x4.9mm_P1.27mm" (id 2) (at 116.84 49.53 0)
-      (effects (font (size 1.27 1.27)) hide)
-    )
+    (property "Footprint" "IC:SOIC-8_3.9x4.9mm_P1.27mm" (id 2) (at 116.84 49.53 0)
+      (effects (font (size 1.27 1.27)) hide)
+    )

Commit message: Bump to board revision B
- Redesign low battery circuit
	- Replace comparator with PMIC
	- Utilize LED Driver IC
	- Remove unneeded 2.5v voltage reference
- Reroute some signals onto wkup/external interrupt pins
Parts:
- removed C24: 1u, Capacitor_SMD:C_0603_1608Metric_Pad1.08x0.95mm_HandSolder, symbol Doorbell_Capacitor:C_Small
- removed D3: BZX84-C8V2,235, Diode_SMD:D_SOT-23_ANK, symbol Doorbell_Diode:D_Zener_Small
- removed Q3: PMPB47XP, Transistor_SMD:PMPB47XP, symbol Doorbell_Transistor_SMD:Q_PMOS_DGS
- removed R21: 2k2, Resistor_SMD:R_0603_1608Metric_Pad0.98x0.95mm_HandSolder, symbol Doorbell_Resistor:R_Small
- removed R24: 180R, Resistor_SMD:R_0805_2012Metric_Pad1.20x1.40mm_HandSolder, symbol Doorbell_Resistor:R_Small
- removed U7: LT6654BHS6-2.5-TRMPBF, IC:LT6654BHS6-2.5-TRMPBF, symbol Doorbell_IC:LT6654BHS6-2.5-TRMPBF
- removed U9: LM2903DR2G, IC:SOIC-8_3.9x4.9mm_P1.27mm, symbol Doorbell_IC:LM2903DR2G
- added Q3: BC847, Transistor_SMD:SOT-23, symbol Doorbell_Transistor_SMD:BC847
- added U7: MAX6457UKD3A+T, IC:MAX6457UKD3A+T, symbol Doorbell_IC:MAX6457UKD3A+T
- added U9: AL5816W5-7, IC:AL5816W5-7, symbol Doorbell_IC:AL5816W5-7
- R17: value 1.8M -> 1M8
- R18: value 1.3M -> 1M; footprint Resistor_SMD:R_0805_2012Metric_Pad1.20x1.40mm_HandSolder -> Resistor_SMD:R_0603_1608Metric_Pad0.98x0.95mm_HandSolder
- R19: value 10M -> 1M; footprint Resistor_SMD:R_0805_2012Metric_Pad1.20x1.40mm_HandSolder -> Resistor_SMD:R_0603_1608Metric_Pad0.98x0.95mm_HandSolder
- R20: value 1M -> 15R; footprint Resistor_SMD:R_0603_1608Metric_Pad0.98x0.95mm_HandSolder -> Resistor_SMD:R_0805_2012Metric_Pad1.20x1.40mm_HandSolder
- R23: value 2k2 -> 2M2
- renumbered R22 to R21
Connections:
- net GND: now also R20.2, Q3.2 (E), U7.2 (GND), U7.4 (~{CLEAR}), U9.2 (GND); no longer R21.2
- net VBAT: now also R19.1, R21.1, R23.1, U7.5 (VCC), U9.5 (Vcc); no longer R17.1, R20.1
- net at U8.5 (EN): now also R19.2, Q3.1 (B), U7.1 (OUT)
- net at R17.2, R18.1: now also U7.3 (IN+); no longer R19.2
- net at R23.2: now also R17.1; no longer R21.1
- net at Q4.1 (B): now also U9.4 (OUT); no longer R23.1
- net at Q4.2 (E): now also R20.1, U9.3 (FB)
- new net: Q3.3 (C), R21.2, U9.1 (PWM)
Other:
- moved on the sheet: C21, C23, D4, Q4, R17, R18, R20, R21
